File: CAD/Circuit Diagrams/KiCAD/ASSI/assi_rounded.kicad_pcb (KiCad board)
At the start: 2 copper layers, 38.1 x 76.2 mm, 24 parts, among them SW2 SW_Push, SW3 SW_Push

Commit message: ASSI PCB mountable
Other:
- board size 38.1 x 76.2 mm -> 48.3 x 76.2 mm
- board text added: "ASSI PCB ver 0.2-RF"
- board text removed: "ASSI PCB ver 0.2-R"

Commit message: Small ASSI PCB fix
Other:
- board text added: "ASSI PCB ver 0.3-RF"
- board text removed: "ASSI PCB ver 0.2-RF"
